File: pcb/hybec-hbl-273-g4/hybec-hbl-273-g4.kicad_pcb (KiCad board)
At the start: 2 copper layers, 24 x 24 mm, 6 parts, among them J1 12V_IN

Commit message: Prepare HYBEC PCB JLCPCB order pack
Other:
- board text added: "JLCJLCJLCJLC"
Changed lines of the file:
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@@
 	(gr_text "HYBEC HBL-273/HBL-667 12V 20W G4" (at 150 110.3 0) (layer "F.Fab") (effects (font (size 0.72 0.72) (thickness 0.10))))
 	(gr_text "non-polar tungsten halogen" (at 150 89.7 0) (layer "F.Fab") (effects (font (size 0.68 0.68) (thickness 0.10))))
+	(gr_text "JLCJLCJLCJLC" (at 150 109.2 0) (layer "B.SilkS") (effects (font (size 0.8 0.8) (thickness 0.10)) (justify mirror)))
 	(segment (start 160 98.46) (end 154.6 98.46) (width 1.2) (layer "F.Cu") (net 1))
 	(segment (start 154.6 98.46) (end 150 98) (width 1.2) (layer "F.Cu") (net 1))
