File: pcb/sk6812rgbw-5050-rgbw-led/sk6812rgbw-5050-rgbw-led.kicad_pcb (KiCad board)
At the start: 2 copper layers, 24 x 24 mm, 8 parts, among them J1 5V_GND_DIN_DOUT

Commit message: Redraw addressable LED carrier boards
Parts:
- removed R1: 330R, Custom:R_0603
- added J2: GND_DIN, Connector_PinHeader_2.54mm:PinHeader_1x02_P2.54mm_Vertical, F.Cu at (158.7, 101.3)
- J1: value 5V_GND_DIN_DOUT -> DOUT_5V; footprint Connector_PinHeader_2.54mm:PinHeader_1x04_P2.54mm_Horizontal -> Connector_PinHeader_2.54mm:PinHeader_1x02_P2.54mm_Vertical; moved to F.Cu
- moved J1 17.6 mm to (141.3, 101.3)
- moved C1 8.46 mm to (150.0, 95.6)
Connections:
- C1 pad 1: GND -> +5V
- C1 pad 2: +5V -> GND
- D1 pad 4: DIN_LED -> DIN
- J1 pad 1: +5V -> DOUT
- J1 pad 2: GND -> +5V
Routing:
- net +5V: track 22.3 -> 9.51 mm
- net GND: track 10.9 -> 22.8 mm
- net DOUT: track 17.5 -> 6.26 mm, vias 1 -> 0
- net DIN: track 1.64 -> 6.26 mm
- net DIN_LED: track 3.05 -> 0.00 mm
Other:
- board text added: "J1: DO/5V J2: G/DI"
- board text removed: "J1: 5V GND DIN DOUT"

Commit message: Clean addressable LED carrier routing
Parts:
- C1: moved to B.Cu
- J1: value DOUT_5V -> 5V_DOUT
- J2: value GND_DIN -> DIN_GND
- moved J1 2.54 mm to (141.3, 98.7)
- moved J2 2.54 mm to (158.7, 98.7)
- moved C1 0.70 mm to (150.0, 96.3)
Connections:
- J1 pad 1: DOUT -> +5V
- J1 pad 2: +5V -> DOUT
- J2 pad 1: GND -> DIN
- J2 pad 2: DIN -> GND
Routing:
- net GND: track 22.8 -> 15.6 mm
- net +5V: track 9.51 -> 14.5 mm
Changed lines of the file:
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@@
 		(fp_line (start 2.75 -2.5) (end -2.75 -2.5) (stroke (width 0.10) (type solid)) (layer "F.Fab"))
 		(fp_rect (start -3.6 -2.85) (end 3.6 2.85) (stroke (width 0.05) (type solid)) (fill none) (layer "F.CrtYd"))
-		(fp_text user "1" (at -4 -1.6 0) (layer "F.SilkS") (effects (font (size 0.8 0.8) (thickness 0.15))))
+		(fp_text user "1" (at -3.65 -3.3 0) (layer "F.SilkS") (effects (font (size 0.8 0.8) (thickness 0.10))))
 		(pad "1" smd roundrect (at -2.45 -1.6) (size 1.5 1.0) (layers "F.Cu" "F.Mask" "F.Paste") (roundrect_rratio 0.08) (net 1 "+5V") (pinfunction "VDD") (pintype "power_in"))
 		(pad "2" smd roundrect (at -2.45 1.6) (size 1.5 1.0) (layers "F.Cu" "F.Mask" "F.Paste") (roundrect_rratio 0.08) (net 4 "DOUT") (pinfunction "DOUT") (pintype "output"))
@@
 	)
 	(footprint "Custom:C_0603"
-		(layer "F.Cu")
-		(at 150 95.6)
-		(descr "0603 capacitor, simple local footprint")
+		(layer "B.Cu")
+		(at 150 96.3)
+		(descr "0603 backside decoupling capacitor, simple local footprint")
 		(property "Reference" "C1"
 			(at 0 -1.1 0)
-			(layer "F.Fab")
+			(layer "B.Fab")
 			(hide yes)
-			(effects (font (size 1 1) (thickness 0.15)))
+			(effects (font (size 1 1) (thickness 0.15)) (justify mirror))
 		)
 		(property "Value" "0.1uF"
 			(at 0 1.1 0)
-			(layer "F.Fab")
-			(effects (font (size 1 1) (thickness 0.15)))
+			(layer "B.Fab")
+			(effects (font (size 1 1) (thickness 0.15)) (justify mirror))
 		)
 		(property "Footprint" "Custom:C_0603"
 			(at 0 0 0)
-			(layer "F.Fab")
+			(layer "B.Fab")
 			(hide yes)
-			(effects (font (size 1 1) (thickness 0.15)))
+			(effects (font (size 1 1) (thickness 0.15)) (justify mirror))
 		)
 		(attr smd)
-		(fp_line (start -0.15 -0.48) (end 0.15 -0.48) (stroke (width 0.10) (type solid)) (layer "F.SilkS"))
-		(fp_line (start -0.15 0.48) (end 0.15 0.48) (stroke (width 0.10) (type solid)) (layer "F.SilkS"))
-		(fp_rect (start -1.55 -0.75) (end 1.55 0.75) (stroke (width 0.05) (type solid)) (fill none) (layer "F.CrtYd"))
-		(fp_rect (start -0.8 -0.4) (end 0.8 0.4) (stroke (width 0.10) (type solid)) (fill none) (layer "F.Fab"))
-		(pad "1" smd roundrect (at -0.8 0) (size 0.8 0.95) (layers "F.Cu" "F.Mask" "F.Paste") (roundrect_rratio 0.15) (net 1 "+5V") (pinfunction "1") (pintype "passive"))
-		(pad "2" smd roundrect (at 0.8 0) (size 0.8 0.95) (layers "F.Cu" "F.Mask" "F.Paste") (roundrect_rratio 0.15) (net 2 "GND") (pinfunction "2") (pintype "passive"))
+		(fp_line (start -0.15 -0.48) (end 0.15 -0.48) (stroke (width 0.10) (type solid)) (layer "B.SilkS"))
+		(fp_line (start -0.15 0.48) (end 0.15 0.48) (stroke (width 0.10) (type solid)) (layer "B.SilkS"))
+		(fp_rect (start -1.55 -0.75) (end 1.55 0.75) (stroke (width 0.05) (type solid)) (fill none) (layer "B.CrtYd"))
+		(fp_rect (start -0.8 -0.4) (end 0.8 0.4) (stroke (width 0.10) (type solid)) (fill none) (layer "B.Fab"))
+		(pad "1" smd roundrect (at -0.8 0) (size 0.8 0.95) (layers "B.Cu" "B.Mask" "B.Paste") (roundrect_rratio 0.15) (net 1 "+5V") (pinfunction "1") (pintype "passive"))
+		(pad "2" smd roundrect (at 0.8 0) (size 0.8 0.95) (layers "B.Cu" "B.Mask" "B.Paste") (roundrect_rratio 0.15) (net 2 "GND") (pinfunction "2") (pintype "passive"))
 	)
 	(footprint "Connector_PinHeader_2.54mm:PinHeader_1x02_P2.54mm_Vertical"
 		(layer "F.Cu")
-		(at 141.3 101.27)
+		(at 141.3 98.73)
 		(descr "Through-hole vertical pin header, 1x02, 2.54mm pitch")
 		(tags "1x02 2.54mm pin header SK6812RGBW clean split")
@@
 			(effects (font (size 1 1) (thickness 0.15)))
 		)
-		(property "Value" "DOUT_5V"
+		(property "Value" "5V_DOUT"
 			(at 0 3.9 0)
 			(layer "F.Fab")
@@
 		)
 		(attr through_hole)
-		(fp_rect (start -1.27 -3.81) (end 1.27 1.27) (stroke (width 0.10) (type solid)) (fill none) (layer "F.Fab"))
-		(fp_rect (start -1.55 -4.1) (end 1.55 1.55) (stroke (width 0.05) (type solid)) (fill none) (layer "F.CrtYd"))
-		(pad "1" thru_hole rect (at 0 0) (size 2.0 2.0) (drill 1.0) (layers "*.Cu" "*.Mask") (remove_unused_layers no) (net 4 "DOUT") (pinfunction "DOUT") (pintype "passive"))
-		(pad "2" thru_hole oval (at 0 -2.54) (size 2.0 2.0) (drill 1.0) (layers "*.Cu" "*.Mask") (remove_unused_layers no) (net 1 "+5V") (pinfunction "5V") (pintype "passive"))
+		(fp_rect (start -1.27 -1.27) (end 1.27 3.81) (stroke (width 0.10) (type solid)) (fill none) (layer "F.Fab"))
+		(fp_rect (start -1.55 -1.55) (end 1.55 4.1) (stroke (width 0.05) (type solid)) (fill none) (layer "F.CrtYd"))
+		(pad "1" thru_hole rect (at 0 0) (size 2.0 2.0) (drill 1.0) (layers "*.Cu" "*.Mask") (remove_unused_layers no) (net 1 "+5V") (pinfunction "5V") (pintype "passive"))
+		(pad "2" thru_hole circle (at 0 2.54) (size 2.0 2.0) (drill 1.0) (layers "*.Cu" "*.Mask") (remove_unused_layers no) (net 4 "DOUT") (pinfunction "DOUT") (pintype "passive"))
 		(model "/usr/share/kicad/3dmodels/Connector_PinHeader_2.54mm.3dshapes/PinHeader_1x02_P2.54mm_Vertical.step" (offset (xyz 0 0 0)) (scale (xyz 1 1 1)) (rotate (xyz 0 0 0)))
 	)
 	(footprint "Connector_PinHeader_2.54mm:PinHeader_1x02_P2.54mm_Vertical"
 		(layer "F.Cu")
-		(at 158.7 101.27)
+		(at 158.7 98.73)
 		(descr "Through-hole vertical pin header, 1x02, 2.54mm pitch")
 		(tags "1x02 2.54mm pin header SK6812RGBW clean split")
@@
 			(effects (font (size 1 1) (thickness 0.15)))
 		)
-		(property "Value" "GND_DIN"
+		(property "Value" "DIN_GND"
 			(at 0 3.9 0)
 			(layer "F.Fab")
@@
 		)
 		(attr through_hole)
-		(fp_rect (start -1.27 -3.81) (end 1.27 1.27) (stroke (width 0.10) (type solid)) (fill none) (layer "F.Fab"))
-		(fp_rect (start -1.55 -4.1) (end 1.55 1.55) (stroke (width 0.05) (type solid)) (fill none) (layer "F.CrtYd"))
-		(pad "1" thru_hole rect (at 0 0) (size 2.0 2.0) (drill 1.0) (layers "*.Cu" "*.Mask") (remove_unused_layers no) (net 2 "GND") (pinfunction "GND") (pintype "passive"))
-		(pad "2" thru_hole oval (at 0 -2.54) (size 2.0 2.0) (drill 1.0) (layers "*.Cu" "*.Mask") (remove_unused_layers no) (net 3 "DIN") (pinfunction "DIN") (pintype "passive"))
+		(fp_rect (start -1.27 -1.27) (end 1.27 3.81) (stroke (width 0.10) (type solid)) (fill none) (layer "F.Fab"))
+		(fp_rect (start -1.55 -1.55) (end 1.55 4.1) (stroke (width 0.05) (type solid)) (fill none) (layer "F.CrtYd"))
+		(pad "1" thru_hole rect (at 0 0) (size 2.0 2.0) (drill 1.0) (layers "*.Cu" "*.Mask") (remove_unused_layers no) (net 3 "DIN") (pinfunction "DIN") (pintype "passive"))
+		(pad "2" thru_hole circle (at 0 2.54) (size 2.0 2.0) (drill 1.0) (layers "*.Cu" "*.Mask") (remove_unused_layers no) (net 2 "GND") (pinfunction "GND") (pintype "passive"))
 		(model "/usr/share/kicad/3dmodels/Connector_PinHeader_2.54mm.3dshapes/PinHeader_1x02_P2.54mm_Vertical.step" (offset (xyz 0 0 0)) (scale (xyz 1 1 1)) (rotate (xyz 0 0 0)))
 	)
@@
 	(gr_text "SK6812RGBW 5050 RGBW" (at 150 110.2 0) (layer "F.Fab") (effects (font (size 0.62 0.62) (thickness 0.10))))
 	(gr_text "J1: DO/5V  J2: G/DI" (at 150 89.8 0) (layer "F.Fab") (effects (font (size 0.52 0.52) (thickness 0.08))))
-	(gr_text "DO" (at 143.55 101.28 0) (layer "F.SilkS") (effects (font (size 0.8 0.8) (thickness 0.11))))
-	(gr_text "5V" (at 143.55 98.72 0) (layer "F.SilkS") (effects (font (size 0.8 0.8) (thickness 0.11))))
-	(gr_text "G" (at 156.55 101.28 0) (layer "F.SilkS") (effects (font (size 0.8 0.8) (thickness 0.11))))
-	(gr_text "DI" (at 156.45 98.72 0) (layer "F.SilkS") (effects (font (size 0.8 0.8) (thickness 0.11))))
+	(gr_text "DO" (at 144 102.75 0) (layer "F.SilkS") (effects (font (size 0.8 0.8) (thickness 0.10))))
+	(gr_text "5V" (at 144 97.25 0) (layer "F.SilkS") (effects (font (size 0.8 0.8) (thickness 0.10))))
+	(gr_text "G" (at 156 102.75 0) (layer "F.SilkS") (effects (font (size 0.8 0.8) (thickness 0.10))))
+	(gr_text "DI" (at 156 97.25 0) (layer "F.SilkS") (effects (font (size 0.8 0.8) (thickness 0.10))))
 	(gr_text "JLCJLCJLCJLC" (at 150 109.2 0) (layer "B.SilkS") (effects (font (size 0.8 0.8) (thickness 0.10)) (justify mirror)))
 	(segment (start 141.3 98.73) (end 147.55 98.4) (width 0.5) (layer "F.Cu") (net 1))
-	(segment (start 147.55 98.4) (end 149.2 95.6) (width 0.35) (layer "F.Cu") (net 1))
-	(segment (start 158.7 101.27) (end 152.45 101.6) (width 0.5) (layer "F.Cu") (net 2))
-	(segment (start 158.7 101.27) (end 160.2 101.27) (width 0.35) (layer "F.Cu") (net 2))
-	(segment (start 160.2 101.27) (end 160.2 95.6) (width 0.35) (layer "F.Cu") (net 2))
-	(segment (start 160.2 95.6) (end 150.8 95.6) (width 0.35) (layer "F.Cu") (net 2))
+	(segment (start 147.55 101.6) (end 141.3 101.27) (width 0.3) (layer "F.Cu") (net 4))
+	(segment (start 152.45 101.6) (end 158.7 101.27) (width 0.5) (layer "F.Cu") (net 2))
 	(segment (start 158.7 98.73) (end 152.45 98.4) (width 0.3) (layer "F.Cu") (net 3))
-	(segment (start 141.3 101.27) (end 147.55 101.6) (width 0.3) (layer "F.Cu") (net 4))
+	(segment (start 149.2 96.3) (end 141.3 98.73) (width 0.35) (layer "B.Cu") (net 1))
+	(segment (start 150.8 96.3) (end 158.7 101.27) (width 0.35) (layer "B.Cu") (net 2))
 )
